Commit message: feat: migrate simulation to Ackermann steering, Zenoh middleware, and hardware-matched sensors
  Replace differential drive with 4-wheel Ackermann steering model matched to the
  real LEGO Bugatti Bolide chassis. Switch from DDS to Zenoh (rmw_zenoh_cpp) and
  update all references from ROS 2 Humble/Gazebo Harmonic to Kilted/Ionic.

  BREAKING CHANGES:
  - angular.z in Twist messages is now a steering angle (rad), not angular velocity
  - Zenoh router (rmw_zenohd) must be running before launching ROS 2 nodes
  - Requires ROS 2 Kilted Kaiju and Gazebo Ionic

  Robot model:
  - Chassis 280x150x100mm, 0.8kg with 4 wheels (radius 21.6mm)
  - Front steering hinge joints (+/-30 deg), rear continuous drive joints
  - gz-sim-ackermann-steering-system plugin replacing libgazebo_ros_diff_drive.so

  Sensors (hardware-matched):
  - Camera: RPi Camera 3 Wide (102 deg HFOV, 1536x864)
  - LIDAR: Slamtec C1 (0.05-12m, 500 samples, 0.03 noise stddev)
  - IMU: BNO085 (gyro 0.054 rad/s, accel 0.3 m/s^2 noise)

  Navigation:
  - compute_steering_angle() with proportional control clamped to max steering
  - Minimum forward speed enforcement (Ackermann cannot pivot)
  - Reduced predictive turn magnitudes and side corrections (0.2 -> 0.1)

File: simulation/urdf/wro_robot.urdf.xacro (robot description, xacro)
@@ -1,12 +1,20 @@
 <?xml version="1.0"?>
 <robot name="wro_robot" xmlns:xacro="http://www.ros.org/wiki/xacro">
-  <!-- Properties -->
-  <xacro:property name="chassis_length" value="0.20"/>
+  <!-- Chassis properties (LEGO Bugatti Bolide) -->
+  <xacro:property name="chassis_length" value="0.28"/>
   <xacro:property name="chassis_width" value="0.15"/>
-  <xacro:property name="chassis_height" value="0.08"/>
-  <xacro:property name="wheel_radius" value="0.035"/>
-  <xacro:property name="wheel_width" value="0.025"/>
-  <xacro:property name="wheel_mass" value="0.1"/>
-  <xacro:property name="chassis_mass" value="1.0"/>
+  <xacro:property name="chassis_height" value="0.10"/>
+  <xacro:property name="chassis_mass" value="0.8"/>
+  <!-- Ackermann geometry -->
+  <xacro:property name="wheelbase" value="0.17"/>
+  <xacro:property name="track_width" value="0.105"/>
+  <xacro:property name="max_steering_angle" value="0.5236"/>
+  <!-- Wheel properties (LEGO Technic wheels) -->
+  <xacro:property name="wheel_radius" value="0.0216"/>
+  <xacro:property name="wheel_width" value="0.020"/>
+  <xacro:property name="wheel_mass" value="0.05"/>
+  <!-- Derived properties -->
+  <xacro:property name="half_wheelbase" value="${wheelbase / 2}"/>
+  <xacro:property name="half_track" value="${track_width / 2}"/>
   <!-- Base link (chassis) -->
   <link name="base_link">
@@ -28,7 +36,9 @@
       <origin xyz="0 0 0" rpy="0 0 0"/>
       <inertia
-        ixx="0.00267" ixy="0.0" ixz="0.0"
-        iyy="0.00417" iyz="0.0"
-        izz="0.00533"/>
+        ixx="${(1.0/12.0) * chassis_mass * (chassis_width*chassis_width + chassis_height*chassis_height)}"
+        ixy="0.0" ixz="0.0"
+        iyy="${(1.0/12.0) * chassis_mass * (chassis_length*chassis_length + chassis_height*chassis_height)}"
+        iyz="0.0"
+        izz="${(1.0/12.0) * chassis_mass * (chassis_length*chassis_length + chassis_width*chassis_width)}"/>
     </inertial>
   </link>
@@ -40,9 +50,98 @@
     <origin xyz="0 0 ${wheel_radius}" rpy="0 0 0"/>
   </joint>
-  <!-- Camera -->
+  <!-- ====== FRONT WHEELS (Steering) ====== -->
+  <!-- Wheel macro for visual/collision/inertial -->
+  <xacro:macro name="wheel_link" params="name">
+    <link name="${name}">
+      <visual>
+        <geometry>
+          <cylinder radius="${wheel_radius}" length="${wheel_width}"/>
+        </geometry>
+        <origin xyz="0 0 0" rpy="${pi/2} 0 0"/>
+        <material name="dark_rubber">
+          <color rgba="0.1 0.1 0.1 1"/>
+        </material>
+      </visual>
+      <collision>
+        <geometry>
+          <cylinder radius="${wheel_radius}" length="${wheel_width}"/>
+        </geometry>
+        <origin xyz="0 0 0" rpy="${pi/2} 0 0"/>
+      </collision>
+      <inertial>
+        <mass value="${wheel_mass}"/>
+        <origin xyz="0 0 0" rpy="${pi/2} 0 0"/>
+        <inertia
+          ixx="${(1.0/12.0) * wheel_mass * (3*wheel_radius*wheel_radius + wheel_width*wheel_width)}"
+          ixy="0.0" ixz="0.0"
+          iyy="${(1.0/12.0) * wheel_mass * (3*wheel_radius*wheel_radius + wheel_width*wheel_width)}"
+          iyz="0.0"
+          izz="${0.5 * wheel_mass * wheel_radius * wheel_radius}"/>
+      </inertial>
+    </link>
+  </xacro:macro>
+  <!-- Steering hinge link (massless) -->
+  <xacro:macro name="steering_link" params="name">
+    <link name="${name}">
+      <inertial>
+        <mass value="0.001"/>
+        <inertia ixx="0.00001" ixy="0.0" ixz="0.0"
+                 iyy="0.00001" iyz="0.0" izz="0.00001"/>
+      </inertial>
+    </link>
+  </xacro:macro>
+  <!-- Front-left steering assembly -->
+  <xacro:steering_link name="front_left_steering"/>
+  <joint name="front_left_steering_joint" type="revolute">
+    <parent link="base_link"/>
+    <child link="front_left_steering"/>
+    <origin xyz="${half_wheelbase} ${half_track} 0" rpy="0 0 0"/>
+    <axis xyz="0 0 1"/>
+    <limit lower="${-max_steering_angle}" upper="${max_steering_angle}" effort="10" velocity="3.0"/>
+  </joint>
+  <xacro:wheel_link name="front_left_wheel"/>
+  <joint name="front_left_wheel_joint" type="continuous">
+    <parent link="front_left_steering"/>
+    <child link="front_left_wheel"/>
+    <origin xyz="0 0 0" rpy="0 0 0"/>
+    <axis xyz="0 1 0"/>
+  </joint>
+  <!-- Front-right steering assembly -->
+  <xacro:steering_link name="front_right_steering"/>
+  <joint name="front_right_steering_joint" type="revolute">
+    <parent link="base_link"/>
+    <child link="front_right_steering"/>
+    <origin xyz="${half_wheelbase} ${-half_track} 0" rpy="0 0 0"/>
+    <axis xyz="0 0 1"/>
+    <limit lower="${-max_steering_angle}" upper="${max_steering_angle}" effort="10" velocity="3.0"/>
+  </joint>
+  <xacro:wheel_link name="front_right_wheel"/>
+  <joint name="front_right_wheel_joint" type="continuous">
+    <parent link="front_right_steering"/>
+    <child link="front_right_wheel"/>
+    <origin xyz="0 0 0" rpy="0 0 0"/>
+    <axis xyz="0 1 0"/>
+  </joint>
+  <!-- ====== REAR WHEELS (Drive) ====== -->
+  <xacro:wheel_link name="rear_left_wheel"/>
+  <joint name="rear_left_wheel_joint" type="continuous">
+    <parent link="base_link"/>
+    <child link="rear_left_wheel"/>
+    <origin xyz="${-half_wheelbase} ${half_track} 0" rpy="0 0 0"/>
+    <axis xyz="0 1 0"/>
+  </joint>
+  <xacro:wheel_link name="rear_right_wheel"/>
+  <joint name="rear_right_wheel_joint" type="continuous">
+    <parent link="base_link"/>
+    <child link="rear_right_wheel"/>
+    <origin xyz="${-half_wheelbase} ${-half_track} 0" rpy="0 0 0"/>
+    <axis xyz="0 1 0"/>
+  </joint>
+  <!-- ====== SENSORS ====== -->
+  <!-- Camera (RPi Camera 3 Wide: 102 deg HFOV, 1536x864) -->
   <link name="camera_link">
     <visual>
       <geometry>
-        <box size="0.025 0.05 0.02"/>
+        <box size="0.024 0.024 0.012"/>
       </geometry>
       <material name="camera_color">
@@ -52,11 +151,11 @@
     <collision>
       <geometry>
-        <box size="0.025 0.05 0.02"/>
+        <box size="0.024 0.024 0.012"/>
       </geometry>
     </collision>
     <inertial>
-      <mass value="0.01"/>
-      <inertia ixx="0.0001" ixy="0.0" ixz="0.0"
-               iyy="0.0001" iyz="0.0" izz="0.0001"/>
+      <mass value="0.005"/>
+      <inertia ixx="0.00001" ixy="0.0" ixz="0.0"
+               iyy="0.00001" iyz="0.0" izz="0.00001"/>
     </inertial>
   </link>
@@ -64,15 +163,14 @@
     <parent link="base_link"/>
     <child link="camera_link"/>
-    <origin xyz="0.08 0 0.05" rpy="0 0.2 0"/>  <!-- Slight downward tilt -->
-  </joint>
-  <!-- Camera sensor (Gazebo plugin) -->
+    <origin xyz="${chassis_length/2 - 0.02} 0 ${chassis_height/2 + 0.01}" rpy="0 0.2 0"/>
+  </joint>
   <gazebo reference="camera_link">
     <sensor name="camera" type="camera">
       <update_rate>30.0</update_rate>
       <camera>
-        <horizontal_fov>2.094</horizontal_fov>  <!-- 120 degrees -->
+        <horizontal_fov>1.7802</horizontal_fov>
         <image>
-          <width>640</width>
-          <height>480</height>
+          <width>1536</width>
+          <height>864</height>
           <format>RGB8</format>
         </image>
@@ -84,5 +182,5 @@
           <type>gaussian</type>
           <mean>0.0</mean>
-          <stddev>0.007</stddev>  <!-- Realistic camera noise -->
+          <stddev>0.007</stddev>
         </noise>
       </camera>
@@ -99,9 +197,9 @@
     </sensor>
   </gazebo>
-  <!-- LiDAR -->
+  <!-- LiDAR (Slamtec C1: 0.05-12m, ~500 samples, 360 deg) -->
   <link name="lidar_link">
     <visual>
       <geometry>
-        <cylinder radius="0.03" length="0.04"/>
+        <cylinder radius="0.0278" length="0.0413"/>
       </geometry>
       <material name="lidar_color">
@@ -111,11 +209,11 @@
     <collision>
       <geometry>
-        <cylinder radius="0.03" length="0.04"/>
+        <cylinder radius="0.0278" length="0.0413"/>
       </geometry>
     </collision>
     <inertial>
-      <mass value="0.05"/>
-      <inertia ixx="0.0001" ixy="0.0" ixz="0.0"
-               iyy="0.0001" iyz="0.0" izz="0.0001"/>
+      <mass value="0.110"/>
+      <inertia ixx="0.00005" ixy="0.0" ixz="0.0"
+               iyy="0.00005" iyz="0.0" izz="0.00004"/>
     </inertial>
   </link>
@@ -123,7 +221,6 @@
     <parent link="base_link"/>
     <child link="lidar_link"/>
-    <origin xyz="0 0 0.06" rpy="0 0 0"/>
-  </joint>
-  <!-- LiDAR sensor (Gazebo plugin) -->
+    <origin xyz="0 0 ${chassis_height/2 + 0.025}" rpy="0 0 0"/>
+  </joint>
   <gazebo reference="lidar_link">
     <sensor name="lidar" type="gpu_ray">
@@ -133,5 +230,5 @@
         <scan>
           <horizontal>
-            <samples>720</samples>
+            <samples>500</samples>
             <resolution>1</resolution>
             <min_angle>-3.14159</min_angle>
@@ -140,5 +237,5 @@
         </scan>
         <range>
-          <min>0.2</min>
+          <min>0.05</min>
           <max>12.0</max>
           <resolution>0.01</resolution>
@@ -147,5 +244,5 @@
           <type>gaussian</type>
           <mean>0.0</mean>
-          <stddev>0.01</stddev>
+          <stddev>0.03</stddev>
         </noise>
       </ray>
@@ -160,10 +257,18 @@
     </sensor>
   </gazebo>
-  <!-- IMU -->
+  <!-- IMU (BNO085) -->
   <link name="imu_link">
+    <visual>
+      <geometry>
+        <box size="0.0256 0.0227 0.0046"/>
+      </geometry>
+      <material name="imu_color">
+        <color rgba="0.0 0.4 0.0 1"/>
+      </material>
+    </visual>
     <inertial>
-      <mass value="0.01"/>
-      <inertia ixx="0.0001" ixy="0.0" ixz="0.0"
-               iyy="0.0001" iyz="0.0" izz="0.0001"/>
+      <mass value="0.0025"/>
+      <inertia ixx="0.00001" ixy="0.0" ixz="0.0"
+               iyy="0.00001" iyz="0.0" izz="0.00001"/>
     </inertial>
   </link>
@@ -177,4 +282,16 @@
       <always_on>true</always_on>
       <update_rate>100.0</update_rate>
+      <imu>
+        <angular_velocity>
+          <x><noise type="gaussian"><mean>0.0</mean><stddev>0.054</stddev></noise></x>
+          <y><noise type="gaussian"><mean>0.0</mean><stddev>0.054</stddev></noise></y>
+          <z><noise type="gaussian"><mean>0.0</mean><stddev>0.054</stddev></noise></z>
+        </angular_velocity>
+        <linear_acceleration>
+          <x><noise type="gaussian"><mean>0.0</mean><stddev>0.3</stddev></noise></x>
+          <y><noise type="gaussian"><mean>0.0</mean><stddev>0.3</stddev></noise></y>
+          <z><noise type="gaussian"><mean>0.0</mean><stddev>0.3</stddev></noise></z>
+        </linear_acceleration>
+      </imu>
       <plugin name="imu_plugin" filename="libgazebo_ros_imu_sensor.so">
         <ros>
@@ -186,142 +303,47 @@
     </sensor>
   </gazebo>
-  <!-- Wheels -->
-  <!-- Left wheel -->
-  <link name="left_wheel">
-    <visual>
-      <geometry>
-        <cylinder radius="${wheel_radius}" length="${wheel_width}"/>
-      </geometry>
-      <origin xyz="0 0 0" rpy="1.5708 0 0"/>
-      <material name="black">
-        <color rgba="0.1 0.1 0.1 1"/>
-      </material>
-    </visual>
-    <collision>
-      <geometry>
-        <cylinder radius="${wheel_radius}" length="${wheel_width}"/>
-      </geometry>
-      <origin xyz="0 0 0" rpy="1.5708 0 0"/>
-    </collision>
-    <inertial>
-      <mass value="${wheel_mass}"/>
-      <origin xyz="0 0 0" rpy="1.5708 0 0"/>
-      <inertia
-        ixx="0.0001" ixy="0.0" ixz="0.0"
-        iyy="0.0001" iyz="0.0" izz="0.0001"/>
-    </inertial>
-  </link>
-  <joint name="left_wheel_joint" type="continuous">
-    <parent link="base_link"/>
-    <child link="left_wheel"/>
-    <origin xyz="0 ${chassis_width/2 + wheel_width/2} 0" rpy="0 0 0"/>
-    <axis xyz="0 1 0"/>
-  </joint>
-  <!-- Right wheel -->
-  <link name="right_wheel">
-    <visual>
-      <geometry>
-        <cylinder radius="${wheel_radius}" length="${wheel_width}"/>
-      </geometry>
-      <origin xyz="0 0 0" rpy="1.5708 0 0"/>
-      <material name="black">
-        <color rgba="0.1 0.1 0.1 1"/>
-      </material>
-    </visual>
-    <collision>
-      <geometry>
-        <cylinder radius="${wheel_radius}" length="${wheel_width}"/>
-      </geometry>
-      <origin xyz="0 0 0" rpy="1.5708 0 0"/>
-    </collision>
-    <inertial>
-      <mass value="${wheel_mass}"/>
-      <origin xyz="0 0 0" rpy="1.5708 0 0"/>
-      <inertia
-        ixx="0.0001" ixy="0.0" ixz="0.0"
-        iyy="0.0001" iyz="0.0" izz="0.0001"/>
-    </inertial>
-  </link>
-  <joint name="right_wheel_joint" type="continuous">
-    <parent link="base_link"/>
-    <child link="right_wheel"/>
-    <origin xyz="0 ${-(chassis_width/2 + wheel_width/2)} 0" rpy="0 0 0"/>
-    <axis xyz="0 1 0"/>
-  </joint>
-  <!-- Caster wheel (front) -->
-  <link name="caster_wheel">
-    <visual>
-      <geometry>
-        <sphere radius="0.02"/>
-      </geometry>
-      <material name="gray">
-        <color rgba="0.5 0.5 0.5 1"/>
-      </material>
-    </visual>
-    <collision>
-      <geometry>
-        <sphere radius="0.02"/>
-      </geometry>
-      <surface>
-        <friction>
-          <ode>
-            <mu>0.0</mu>
-            <mu2>0.0</mu2>
-          </ode>
-        </friction>
-      </surface>
-    </collision>
-    <inertial>
-      <mass value="0.01"/>
-      <inertia ixx="0.00001" ixy="0.0" ixz="0.0"
-               iyy="0.00001" iyz="0.0" izz="0.00001"/>
-    </inertial>
-  </link>
-  <joint name="caster_wheel_joint" type="fixed">
-    <parent link="base_link"/>
-    <child link="caster_wheel"/>
-    <origin xyz="0.07 0 -0.025" rpy="0 0 0"/>
-  </joint>
-  <!-- Differential drive controller -->
+  <!-- ====== ACKERMANN STEERING CONTROLLER ====== -->
   <gazebo>
-    <plugin name="diff_drive_controller" filename="libgazebo_ros_diff_drive.so">
-      <ros>
-        <namespace>/wro_robot</namespace>
-      </ros>
-      <!-- Wheels -->
-      <left_joint>left_wheel_joint</left_joint>
-      <right_joint>right_wheel_joint</right_joint>
-      <!-- Kinematics -->
-      <wheel_separation>${chassis_width + wheel_width}</wheel_separation>
-      <wheel_diameter>${2*wheel_radius}</wheel_diameter>
-      <!-- Limits -->
-      <max_wheel_torque>2.0</max_wheel_torque>
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