Commit message: chore(robot): sync physical vehicle specifications and sensor mount architectures
Overhaul physical specifications across the monorepo to align with real-world
vehicle dimensions, resolve chassis structural drift, and correct sensor transforms.

- Update canonical vehicle specs: increase TRACK_WIDTH to 0.1675m, WHEELBASE to
  0.19m, WHEEL_RADIUS to 0.035m, and WHEEL_WIDTH to 0.025m.
- Introduce explicit sensor installation offsets: apply LIDAR_MOUNT_X_OFFSET (0.1222m)
  and adjust CAMERA_MOUNT_X/Z_OFFSET positions to match true physical configurations.
- Propagate specs consistently to clear duplication across subsystems: update real-robot
  URDF/Xacro models, static TF launch configurations, the wheel-encoder driver,
  and test assertions.
- Resolve a structural drift bug in the Go-based Gazebo simulation generator
  by correcting stale 0.28x0.15m chassis bounding-box overrides to the current
  0.30x0.20m geometry standard.
- Implement camera down-tilt support (CAMERA_MOUNT_PITCH_DEG=30) across TF and URDF
  definition pipelines.
- Generate a canonical tracking matrix (`docs/robot-physical-constants.md`) mapping
  the file:line coordinate bounds of all structural parameters across Python and Go.
- Flag a pending 3D pinhole camera projection coordinate fix inside the sign-routing logic.

File: platform/gazebo/runtime/robot_description/wro_robot.urdf.xacro (robot description, xacro)
@@ -1,17 +1,28 @@
 <?xml version="1.0"?>
 <robot name="wro_robot" xmlns:xacro="http://www.ros.org/wiki/xacro">
-  <!-- Chassis properties (LEGO Bugatti Bolide) -->
-  <xacro:property name="chassis_length" value="0.28"/>
-  <xacro:property name="chassis_width" value="0.15"/>
+  <!-- Chassis properties (LEGO Bugatti Bolide) -- measured 2026-07-11, see
+       ../../../robot/docs/robot-physical-constants.md. Must match
+       platform/shared/src/shared/config/constants.py's RobotSpecs -- kept in sync by hand,
+       there is no single source of truth across Python/xacro/the Go SDF generator yet. -->
+  <xacro:property name="chassis_length" value="0.30"/>
+  <xacro:property name="chassis_width" value="0.20"/>
   <xacro:property name="chassis_height" value="0.10"/>
   <xacro:property name="chassis_mass" value="0.8"/>
   <!-- Ackermann geometry -->
-  <xacro:property name="wheelbase" value="0.17"/>
-  <xacro:property name="track_width" value="0.105"/>
+  <xacro:property name="wheelbase" value="0.19"/>
+  <xacro:property name="track_width" value="0.1675"/>
   <xacro:property name="max_steering_angle" value="0.5236"/>
-  <!-- Wheel properties (LEGO Technic wheels) -->
-  <xacro:property name="wheel_radius" value="0.0216"/>
-  <xacro:property name="wheel_width" value="0.020"/>
+  <!-- Wheel properties -->
+  <xacro:property name="wheel_radius" value="0.035"/>
+  <xacro:property name="wheel_width" value="0.025"/>
   <xacro:property name="wheel_mass" value="0.05"/>
+  <!-- Sensor mount offsets. lidar_mount_x = chassis_length/2 - lidar_link's own mesh radius
+       (0.0278, see below): the C1 mounted flush with the front edge. camera_mount_x/z/pitch
+       are an estimate pending a real measurement -- see RobotSpecs.CAMERA_MOUNT_* in
+       constants.py. Must match RobotSpecs.LIDAR_MOUNT_X_OFFSET / CAMERA_MOUNT_*. -->
+  <xacro:property name="lidar_mount_x" value="0.1222"/>
+  <xacro:property name="camera_mount_x" value="0.1222"/>
+  <xacro:property name="camera_mount_z" value="0.16"/>
+  <xacro:property name="camera_mount_pitch" value="0.5236"/>  <!-- ~30 degrees, tilted down -->
   <!-- Derived properties -->
   <xacro:property name="half_wheelbase" value="${wheelbase / 2}"/>
@@ -163,5 +174,5 @@
     <parent link="base_link"/>
     <child link="camera_link"/>
-    <origin xyz="${chassis_length/2 - 0.02} 0 ${chassis_height/2 + 0.01}" rpy="0 0.2 0"/>
+    <origin xyz="${camera_mount_x} 0 ${camera_mount_z}" rpy="0 ${camera_mount_pitch} 0"/>
   </joint>
   <gazebo reference="camera_link">
@@ -221,5 +232,5 @@
     <parent link="base_link"/>
     <child link="lidar_link"/>
-    <origin xyz="0 0 ${chassis_height/2 + 0.025}" rpy="0 0 0"/>
+    <origin xyz="${lidar_mount_x} 0 ${chassis_height/2 + 0.025}" rpy="0 0 0"/>
   </joint>
   <gazebo reference="lidar_link">

Commit message: chore(robot): inject vehicle visualization markers into rviz and verify sensor pitch
Enhance the closed-loop simulation visualizer to support localized geometric testing,
and validate physical camera pitch transforms via RViz rendering engines.

- Implement real-time vehicle footprint and sensor layout markers (chassis box,
  LIDAR cylinder, and a directional camera orientation arrow) inside `live_visualizer.py`.
- Resolve a marker race condition under volatile RViz QoS configurations by switching
  from a one-shot publish sequence to a 1Hz periodic republish loop.
- Rectify a joint transform mismatch in `wro_robot.urdf.xacro`, aligning the `lidar_joint`
  vertical z-offset (0.12m) across all physical specification targets.
- Graphically verify the directional sign parity of `CAMERA_MOUNT_PITCH_DEG=30` (confirming
  a true down-and-forward projection angle).
- Document layout confirmations and visual mapping frameworks inside the reference index
  (`docs/robot-physical-constants.md`) while delineating structural mechanical pitch profiles
  from dynamic inertial IMU orientation streams.

File: platform/gazebo/runtime/robot_description/wro_robot.urdf.xacro (robot description, xacro)
@@ -232,5 +232,10 @@
     <parent link="base_link"/>
     <child link="lidar_link"/>
-    <origin xyz="${lidar_mount_x} 0 ${chassis_height/2 + 0.025}" rpy="0 0 0"/>
+    <!-- z = chassis_height + 0.02 = 0.12: matches static_tfs.launch.py / the Go SDF
+         generator's RobotHeight + RobotLidarZOffset. Previously chassis_height/2 + 0.025
+         = 0.075 here only -- a pre-existing drift from those other two sources, found
+         and fixed alongside the mount-offset measurements (see
+         platform/robot/docs/robot-physical-constants.md). -->
+    <origin xyz="${lidar_mount_x} 0 ${chassis_height + 0.02}" rpy="0 0 0"/>
   </joint>
   <gazebo reference="lidar_link">

Commit message: feat(robot): implement centralized toml single source of truth and go robot-constants generator
Consolidate physical vehicle metrics and mounting vectors into a single source of truth,
building a programmatic Go generation pipeline to coordinate Python, Go, and xacro layouts.

- Configuration: Author `platform/shared/config/robot.toml` to serve as the unified structural
  matrix for chassis, Ackermann kinematics, and camera/LIDAR offsets.
- Generator Subsystem: Extend the `simgen` Go CLI utility with a `generate-robot-constants`
  subcommand using the new `internal/robotconfig` package to process values cleanly.
- Target Outputs: Output programmatic files with `DO NOT EDIT` headers—including a gofmt-formatted
  `robot_constants.gen.go`, a `robot_properties.gen.xacro` declaration snippet, and an isolated
  `robot_constants_gen.py` Python library.
- Consumer Wiring: Strip legacy hardcoded references from `constants.go`, adapt `wro_robot.urdf.xacro`
  via inclusion hooks, and refactor the core Python `RobotSpecs` layout block.
- Verification: Fix independent value tracking duplicates inside `test_constants.py`, pass
  all 307 backend unit tests, and secure clean formatting checks across ruff and golangci-lint.

File: platform/gazebo/runtime/robot_description/wro_robot.urdf.xacro (robot description, xacro)
@@ -1,28 +1,7 @@
 <?xml version="1.0"?>
 <robot name="wro_robot" xmlns:xacro="http://www.ros.org/wiki/xacro">
-  <!-- Chassis properties (LEGO Bugatti Bolide) -- measured 2026-07-11, see
-       ../../../robot/docs/robot-physical-constants.md. Must match
-       platform/shared/src/shared/config/constants.py's RobotSpecs -- kept in sync by hand,
-       there is no single source of truth across Python/xacro/the Go SDF generator yet. -->
-  <xacro:property name="chassis_length" value="0.30"/>
-  <xacro:property name="chassis_width" value="0.20"/>
-  <xacro:property name="chassis_height" value="0.10"/>
-  <xacro:property name="chassis_mass" value="0.8"/>
-  <!-- Ackermann geometry -->
-  <xacro:property name="wheelbase" value="0.19"/>
-  <xacro:property name="track_width" value="0.1675"/>
-  <xacro:property name="max_steering_angle" value="0.5236"/>
-  <!-- Wheel properties -->
-  <xacro:property name="wheel_radius" value="0.035"/>
-  <xacro:property name="wheel_width" value="0.025"/>
-  <xacro:property name="wheel_mass" value="0.05"/>
-  <!-- Sensor mount offsets. lidar_mount_x = chassis_length/2 - lidar_link's own mesh radius
-       (0.0278, see below): the C1 mounted flush with the front edge. camera_mount_x/z/pitch
-       are an estimate pending a real measurement -- see RobotSpecs.CAMERA_MOUNT_* in
-       constants.py. Must match RobotSpecs.LIDAR_MOUNT_X_OFFSET / CAMERA_MOUNT_*. -->
-  <xacro:property name="lidar_mount_x" value="0.1222"/>
-  <xacro:property name="camera_mount_x" value="0.1222"/>
-  <xacro:property name="camera_mount_z" value="0.16"/>
-  <xacro:property name="camera_mount_pitch" value="0.5236"/>  <!-- ~30 degrees, tilted down -->
+  <!-- Chassis/Ackermann/wheel/sensor-mount properties -- generated from
+       platform/shared/config/robot.toml, see robot_properties.gen.xacro. -->
+  <xacro:include filename="robot_properties.gen.xacro"/>
   <!-- Derived properties -->
   <xacro:property name="half_wheelbase" value="${wheelbase / 2}"/>
