Commit message: fix(state): require vision only for the Obstacle Challenge
all_ready gated on hailo_ready unconditionally, so an unloaded Hailo model
blocked BOOT_CHECK for BOTH challenges -- the robot could not start a race at
all without vision. But traffic signs only exist in the Obstacle Challenge;
the Open Challenge navigates on LIDAR alone, so vision is dead weight there.

That matters now rather than later: the YOLOv11->Hailo conversion is still
pending, and this was the only thing preventing Open Challenge runs on real
hardware -- which is also the simpler mode for validating the navigation
changes made today (steer_kp, counter-phase geometry, closed-loop speed).

challenge_mode is latched earlier in BOOT_CHECK so it is known here, and
while it is still None the challenge_mode_status term keeps readiness false
anyway, so treating vision as required until then is safe. The per-tick
"Hailo not ready" warning is likewise suppressed in Open, where it would
report a blocker that blocks nothing.

File: platform/gazebo/runtime/robot_description/robot_properties.gen.xacro (robot description, xacro)
@@ -10,5 +10,5 @@
   <xacro:property name="wheelbase" value="0.19"/>
   <xacro:property name="track_width" value="0.1675"/>
-  <xacro:property name="max_steering_angle" value="0.5236"/>
+  <xacro:property name="max_steering_angle" value="1.2253"/>
   <!-- Wheel properties -->
   <xacro:property name="wheel_radius" value="0.035"/>

Commit message: refactor(robot): centralize hardware and navigation config in TOML
Cause

Hardware driver and navigation-tuning defaults were scattered across
module-level constants, dataclass field defaults, and .env.example --
three different places to check for the same value, with no single
source of truth and env vars that silently did nothing for most
drivers because nothing read them. This also blocked answering "what
does this robot actually run with" without reading source.

Key Changes

Hardware config (Tier 2)
- Add src/hardware/settings_base.py: HardwareBaseSettings, a shared
  pydantic-settings base that reads config/hardware/**/*.toml, with
  an env var of the same name still overriding the TOML value.
- Migrate 14 remaining hardware Config classes to it: camera (config,
  rpicam driver, rpi camera_module_3 driver), hailo (Config +
  StreamingConfig), button (gpio, mcp2221), teleop, motors (Config +
  ServoConfig), challenge_mode, and all four bno08x IMU variants
  (plain + mcp2221, i2c + uart_rvc). ssd1306/oled_display_node's
  NodeConfig were already migrated as the pilot.
- Add matching TOML files under config/hardware/**/. Fields with no
  known real value (device ports, GPIO pins never documented in
  .env.example) are deliberately left out, required from env exactly
  as before this migration -- same fail-closed behavior, just visible
  now via the TOML file's own comment instead of silent.

Navigation config (Tier 3)
- NavigationTuning now loads from platform/shared/config/navigation/
  *.toml (12 groups: clearance, heading, pursuit, speed, escape,
  sensor, waypoints, lidar_sectors, sign_router, sign_discovery,
  parking, localization).
- CollisionAvoidanceController, WaypointController, SignRouter,
  ObservedSignMap, ParkController, and LidarLocalizer now take these
  values as constructor params instead of reading module constants.
- Fixes two dead-default bugs this uncovered: steer_kp (1.5 -> 1.2)
  and fast_dist (0.50 -> 1.00) were never actually reachable from the
  old module-constant wiring.
- shared/domain/models.py gains the typed models this wiring threads
  through consumers (gateway.py, track_model.py, node.py,
  vision_emulator.py, race_tracker.py's LoopProgress, corridor
  geometry/width measurements) instead of passing raw dicts/tuples.

Vision config (Tier 4)
- DetectorConfig (src/vision/detector.py) migrated to
  HardwareBaseSettings for min_confidence/output_format; model_path
  and class_to_color stay caller-supplied (backend-specific/derived),
  matching every existing call site.
- VisionNode (src/ros2/vision/node.py) gains a Config class sourcing
  its declare_parameter defaults from config/hardware/vision/node.toml,
  while keeping every declare_parameter/get_parameter call so
  rpi5_nodes.launch.py's launch-time overrides (backend, model_path,
  camera_source, publish_annotated, publish_raw) keep working exactly
  as before -- TOML only changes the fallback when no override is set.

.env.example trim
- Cut from 307 to 146 lines: removed every var that now has a TOML
  default, keeping only fields with no TOML default (device ports),
  values read directly by launch files/nodes outside the TOML system
  (HAILO_MODEL_PATH, VISION_DEBUG_VIDEO), and genuine runtime/ops
  knobs unrelated to any driver (motor backend selection, DC-encoder
  pins not yet migrated, sensor/IP timeouts, race/ROS2/logging config).

Also bundled in (found during hardware verification of the above)
- telemetry_bridge_node.py: /system_status publisher is now
  TRANSIENT_LOCAL (matching state_machine_node's), and
  ui_summary_rate_hz default raised 2Hz -> 10Hz to match the OLED's
  own redraw rate.
- oled_display_node.py: /system_status subscription now requests the
  matching latched QoS, since the publisher-side fix above makes that
  safe (previously the subscriber had to stay VOLATILE to remain
  QoS-compatible with a VOLATILE publisher, so it could never get the
  current value from a late/restarted publisher).
- collision_avoidance_controller.py: _sector_ranges now excludes
  non-finite (inf, no-return) LIDAR rays from its mask. A single
  no-return ray landing inside a sector's angular window previously
  poisoned that sector's mean/min/max to infinity -- affecting both
  the OLED's displayed clearances and detect_threat_direction's real
  collision-avoidance sectors.

Verification

- Full test suite on real Pi 5 hardware: 641 passed, 15 pre-existing
  failures unrelated to this work (confirmed against git history).
- All 15 migrated hardware Config classes smoke-tested (import +
  instantiate with real .env values) on Pi 5; 12 succeed outright, the
  3 that don't are documented pre-existing gaps (picamera2 missing
  from the pixi env, two IMU/button variants not currently deployed
  and never given real values in .env.example either, before or after
  this migration).
- Deployed and verified live: state machine reaches BOOT_CHECK ->
  READY cleanly, OLED shows correct real-time telemetry (no more
  stale display after a Pi 5 restart), vision node runs at 15fps on
  the Hailo NPU.

File: platform/gazebo/runtime/robot_description/robot_properties.gen.xacro (robot description, xacro)
@@ -17,4 +17,5 @@
   <!-- Sensor mount offsets -->
   <xacro:property name="lidar_mount_x" value="0.1222"/>
+  <xacro:property name="lidar_mount_yaw_offset_deg" value="180"/>
   <xacro:property name="camera_mount_x" value="0.1222"/>
   <xacro:property name="camera_mount_z" value="0.16"/>

Commit message: refactor(robot,gazebo): promote LIDAR/IMU mount z-offsets into robot.toml
Cause: platform audit item 23 flagged static_tfs.launch.py's hardcoded
0.12/0.01 LIDAR/IMU z-offsets. Investigation found these values already
existed as hand-written Go constants (simconfig.RobotLidarZOffset=0.02,
RobotImuZOffset=0.01, not generated from robot.toml) that the SDF
generator correctly used, while static_tfs.launch.py and the URDF xacro
each separately hardcoded the same facts as literals -- three
independent copies of the same two numbers.

While tracing all three copies, found a real bug: the URDF xacro's
imu_link joint hardcoded z=0 instead of 0.01, so the IMU was actually
misplaced in RViz/the URDF tree (the SDF generator and static_tfs.launch.py
both had the correct 0.01; only the xacro was wrong).

Key Changes:
- shared/config/robot.toml: added lidar.mount_z_offset and a new [imu]
  section with mount_z_offset, matching the existing camera mount-offset
  pattern
- robotconfig/{config,generate}.go: parse the two new TOML fields, emit
  RobotLidarMountZOffset/RobotImuMountZOffset (Go), lidar_mount_z/
  imu_mount_z (xacro properties), LIDAR_MOUNT_Z_OFFSET/IMU_MOUNT_Z_OFFSET
  (Python) -- ran through the real `task gen:robot-constants` generator,
  not hand-edited
- simconfig/constants.go: removed the now-redundant hand-written
  RobotLidarZOffset/RobotImuZOffset; sdf/robot.go's two call sites
  updated to the generated names
- wro_robot.urdf.xacro: lidar_joint now uses ${lidar_mount_z} instead of
  a bare 0.02 literal; imu_joint fixed to use ${imu_mount_z} instead of
  the wrong hardcoded 0
- shared/config/constants.py (RobotSpecs): expose LIDAR_MOUNT_Z_OFFSET
  and IMU_MOUNT_Z_OFFSET from the generated module, matching the
  existing camera mount-offset fields
- static_tfs.launch.py: replaced the 0.12/0.01 literals with
  RobotSpecs.HEIGHT + RobotSpecs.LIDAR_MOUNT_Z_OFFSET and
  RobotSpecs.IMU_MOUNT_Z_OFFSET

Verification:
- Regenerated all 3 consumers via `task gen:robot-constants`; diffs are
  purely additive, confirming the hand-bootstrapped Go constant (needed
  to break the build<->generate circular dependency) matched what the
  generator itself produces
- Computed static_tfs.launch.py's new derived values: LIDAR z = 0.12,
  IMU z = 0.01 -- identical to the old hardcoded literals
- go build/vet/test and golangci-lint clean across
  platform/gazebo/generator (only a pre-existing, untouched golines
  finding elsewhere in the same file)
- shared.config.navigation_tuning test suite still passes (constants.py
  still imports and constructs correctly)

File: platform/gazebo/runtime/robot_description/robot_properties.gen.xacro (robot description, xacro)
@@ -17,5 +17,7 @@
   <!-- Sensor mount offsets -->
   <xacro:property name="lidar_mount_x" value="0.1222"/>
+  <xacro:property name="lidar_mount_z" value="0.02"/>
   <xacro:property name="lidar_mount_yaw_offset_deg" value="180"/>
+  <xacro:property name="imu_mount_z" value="0.01"/>
   <xacro:property name="camera_mount_x" value="0.1222"/>
   <xacro:property name="camera_mount_z" value="0.16"/>

File: platform/gazebo/runtime/robot_description/wro_robot.urdf.xacro (robot description, xacro)
@@ -211,10 +211,11 @@
     <parent link="base_link"/>
     <child link="lidar_link"/>
-    <!-- z = chassis_height + 0.02 = 0.12: matches static_tfs.launch.py / the Go SDF
-         generator's RobotHeight + RobotLidarZOffset. Previously chassis_height/2 + 0.025
-         = 0.075 here only -- a pre-existing drift from those other two sources, found
-         and fixed alongside the mount-offset measurements (see
-         platform/robot/docs/robot-physical-constants.md). -->
-    <origin xyz="${lidar_mount_x} 0 ${chassis_height + 0.02}" rpy="0 0 0"/>
+    <!-- z = chassis_height + lidar_mount_z = 0.12: matches static_tfs.launch.py / the Go
+         SDF generator's RobotHeight + RobotLidarMountZOffset. Previously chassis_height/2
+         + 0.025 = 0.075 here only -- a pre-existing drift from those other two sources,
+         found and fixed alongside the mount-offset measurements (see
+         platform/robot/docs/robot-physical-constants.md). lidar_mount_z is now generated
+         from platform/shared/config/robot.toml (was a hardcoded 0.02 literal here). -->
+    <origin xyz="${lidar_mount_x} 0 ${chassis_height + lidar_mount_z}" rpy="0 0 0"/>
   </joint>
   <gazebo reference="lidar_link">
@@ -271,5 +272,9 @@
     <parent link="base_link"/>
     <child link="imu_link"/>
-    <origin xyz="0 0 0" rpy="0 0 0"/>
+    <!-- z = imu_mount_z = 0.01: matches static_tfs.launch.py / the Go SDF generator's
+         RobotImuMountZOffset. Was hardcoded to 0 here only -- a pre-existing drift from
+         those other two sources, found while consolidating the mount-offset source of
+         truth into platform/shared/config/robot.toml. -->
+    <origin xyz="0 0 ${imu_mount_z}" rpy="0 0 0"/>
   </joint>
   <gazebo reference="imu_link">

Commit message: refactor(config): give the mat, the robot and the tuning one source each
The mat's geometry was maintained twice by hand -- once in the Python classes
of shared/config/constants.py, once in the Go const blocks of
simconfig/constants.go, whose header asked future editors to keep the two in
sync themselves. Around forty tuning values had the same shape: a literal in
the module beside a comment naming the config field it duplicated.

That arrangement had already failed, quietly, in three places. The sign
router's DEFORM_DEPTH_BUFFER_M sat in its TOML with no reader at all while a
duplicate literal did the work. tests/test_constants.py carried
SIGN_ACTIVATION_DIST 0.80 and SIGN_PASSED_DIST 1.20 against a router retuned to
1.40 and 1.60 -- and the robot positions in test_sign_router.py were written as
raw distances chosen against the old pair, so "drive 1.5 m past it" silently
stopped meaning past and no test changed. Comments are not a mechanism.

track.toml now joins robot.toml as a generated source of truth: `task
gen:track-constants` renders it into Go and Python, and the hand-written
duplicates are gone. Its derived values are computed in exact decimal
arithmetic rather than float64, because 0.60 - 0.40 evaluates to
0.19999999999999996 and a generator that emitted that would be writing
representation error into the file meant to be authoritative. Four constants
holding two numbers -- the corridor division lines, restated as the sign grid's
lanes -- collapse into one declaration the rest derive from.

The starting geometry was wrong, not merely duplicated. simgen placed the robot
at 0.3/0.5/0.7 of the corridor width, which emits six positions whatever the
width, straddles a band boundary at 0.42 in a narrow corridor, and never emits
a start against the inner block. The mat's real layout is bands of 40/20/40 cm
out from the outer wall, so a narrow corridor holds four legal cells and a wide
one six. The spawn is now the chassis pushed flush against a named band edge
and derived from its measured width, never centred: one band edge is a painted
line the robot may sit against harmlessly, the other may be the block, so
splitting the slack spends half the margin on the line. NavigationTuning also
refuses to load a config where the corner turn begins before the direction
window opens -- a cross-file invariant that no single TOML could see.

Chassis width is 0.194 m, not 0.20, and the assembled car weighs 1.5 kg, not
1.0. Both were re-measured; mass reaches the inertia tensors, so it is not
bookkeeping.

Two things this leaves open. The narrow corridor's middle band is a legal start
that fails 23 times out of 23, under both contact policies and at the corrected
width -- the robot cannot free itself from a wall it begins against, which is
almost certainly the same defect as the four red deviation-recovery cases. And
the fixtures never contained that start, which is exactly why every sweep to
date read clean.

This should have been several commits. It is one because the work was done
against a working tree that already held it.

File: platform/gazebo/runtime/robot_description/robot_properties.gen.xacro (robot description, xacro)
@@ -2,9 +2,9 @@
 <!-- Code generated by `simgen generate-robot-constants` from platform/shared/config/robot.toml. DO NOT EDIT. -->
 <robot xmlns:xacro="http://www.ros.org/wiki/xacro">
-  <!-- Chassis properties (LEGO Bugatti Bolide) -->
+  <!-- Chassis properties (vTitan) -->
   <xacro:property name="chassis_length" value="0.3"/>
-  <xacro:property name="chassis_width" value="0.2"/>
+  <xacro:property name="chassis_width" value="0.194"/>
   <xacro:property name="chassis_height" value="0.1"/>
-  <xacro:property name="chassis_mass" value="0.8"/>
+  <xacro:property name="chassis_mass" value="1.3"/>
   <!-- Ackermann geometry -->
   <xacro:property name="wheelbase" value="0.19"/>
@@ -18,5 +18,5 @@
   <xacro:property name="lidar_mount_x" value="0.1222"/>
   <xacro:property name="lidar_mount_z" value="0.02"/>
-  <xacro:property name="lidar_mount_yaw_offset_deg" value="180"/>
+  <xacro:property name="lidar_mount_yaw_offset_deg" value="180.0"/>
   <xacro:property name="imu_mount_z" value="0.01"/>
   <xacro:property name="camera_mount_x" value="0.1222"/>

Commit message: fix(robot): derive the steering limit instead of stating it in four places
The road-wheel angle at full lock was written down four times, and three of
them disagreed.

motors.toml had the two measured facts: the servo reaches 90 degrees of travel
and the linkage produces 0.78 road-wheel degrees per servo degree. robot.toml
had their product, 1.2253 rad, computed by hand, under a comment saying the
factors lived in .env.example -- which by then said to see motors.toml. And the
code defaults said something else entirely: MotorSteeringConfig defaulted to 45
degrees at a 1.0 ratio, which is not this chassis but a direct-drive one with
half the travel, while WaypointController defaulted to 0.5236 rad -- the ~30
degree value robot.toml's own comment says understated the chassis by more than
half.

Nothing was broken in practice only because motors.toml is present and
overrides the defaults. A deployment without it, or a unit constructing
WaypointController directly, gets a planner that believes the robot turns half
as sharply as it does.

The two measured facts move to robot.toml, where the rest of the chassis is,
and the limit is derived from them at generation time. motors.toml stops
declaring them and says why; per-unit overrides stay available through
MOTOR_STEERING__*. The generated value is now 1.2252211349 rather than the
rounded 1.2253 -- 0.0045 degrees, but arrived at rather than typed.

Also fixes the generator's own remaining decimal-point bug, the one already
fixed in trackconfig: MAX_ACCEL_MPS2 was emitted as `2`, which Python binds as
an int under a Final[float] annotation.

File: platform/gazebo/runtime/robot_description/robot_properties.gen.xacro (robot description, xacro)
@@ -10,5 +10,5 @@
   <xacro:property name="wheelbase" value="0.19"/>
   <xacro:property name="track_width" value="0.1675"/>
-  <xacro:property name="max_steering_angle" value="1.2253"/>
+  <xacro:property name="max_steering_angle" value="1.2252211349000193"/>
   <!-- Wheel properties -->
   <xacro:property name="wheel_radius" value="0.035"/>

Commit message: fix(shared): declare bench-measured max_wheel_angle_deg instead of a stale linkage_ratio
Cause: robot.toml's [steering] linkage_ratio = 0.78 (90 deg servo -> ~70.2
deg wheel) was never re-measured after the linkage geometry changed and had
drifted. A 2026-08-09 bag analysis found a ~1.8x global under-turn on
hardware and flagged linkage_ratio as one of two untested candidates,
recommending a bench measurement with a protractor instead of guessing from
bag data. Done 2026-08-10: with the servo at its true 90 deg end-stop
(confirmed not stalling early), the front wheel reaches only ~55 deg.

A bare ratio is also awkward to re-measure and re-declare by hand each time
the linkage or servo changes, so the source-of-truth field is now the
bench-measured angle itself; the ratio is derived from it wherever a
consumer still wants that form.

Key Changes:
- robot.toml: [steering] now declares max_wheel_angle_deg = 55.0 instead of
  linkage_ratio = 0.78
- robotconfig/config.go: Steering.MaxWheelAngleDeg replaces LinkageRatio;
  added a LinkageRatio() method derived from it, and simplified
  MaxSteeringAngle() to convert MaxWheelAngleDeg directly
- robotconfig/generate.go: emits RobotMaxWheelAngleDeg plus a derived
  RobotLinkageRatio into the generated Go constants
- robot_constants.gen.go / robot_properties.gen.xacro: regenerated via
  `task gen:robot-constants` -- RobotMaxSteering 1.2252 rad (70.2 deg) ->
  0.9599 rad (55 deg)
- shared/config/robot_constants.py: Steering.max_wheel_angle_deg is the
  declared field; linkage_ratio and max_steering_angle are now derived
  properties
- shared/config/constants/robot.py: added RobotSpecs.MAX_WHEEL_ANGLE_DEG;
  LINKAGE_RATIO and MAX_STEERING_ANGLE stay as Final constants so no
  existing consumer (ackermann_motor_node.py, diag_bag_steer.py, test
  mocks) needed to change

Verification: `task gen:robot-constants` regenerated cleanly; Python
RobotConstants.load_default() and RobotSpecs confirmed to load
max_wheel_angle_deg=55.0, linkage_ratio=0.6111 correctly. Not
hardware-validated beyond the bench protractor reading itself -- this only
closes a 1.28x correction of the 1.82x under-turn the bag data measured, so
the crosstrack drift is not confirmed fixed; re-run
diag_bag_steer.py --effectiveness on fresh hardware bags before declaring
it resolved.

File: platform/gazebo/runtime/robot_description/robot_properties.gen.xacro (robot description, xacro)
@@ -10,5 +10,5 @@
   <xacro:property name="wheelbase" value="0.19"/>
   <xacro:property name="track_width" value="0.1675"/>
-  <xacro:property name="max_steering_angle" value="1.2252211349000193"/>
+  <xacro:property name="max_steering_angle" value="0.9599310885968813"/>
   <!-- Wheel properties -->
   <xacro:property name="wheel_radius" value="0.035"/>
