Commit message: fix(sim): make the Gazebo URDF a counter-phase 4WS car, and parseable at all
The robot description had two independent defects, both committed and
neither covered by a test. It did not parse, and if it had, it described a
front-steer car rather than the counter-phase four-wheel-steer chassis the
headless sim and the real robot both are.

Cause:
1. Three XML comments contained `--`, which is illegal inside a comment.
   xacro raised ExpatError on line 4, so every launch depending on the robot
   description was dead. Nothing caught it because nothing expanded the file
   -- Gazebo is the only consumer, and it is not exercised by any test.
2. The rear wheels were plain `continuous` joints bolted straight to
   base_link. Counter-phase moves the instantaneous centre of rotation from
   the rear axle to the chassis centre (L_eff = wheelbase / (1 + ratio)), so
   the robot yaws TWICE as fast at a given steering angle. This is the same
   defect already found and fixed once in src/simulation/kinematics.py,
   where it had silently made every gain tuned against the sim hotter on the
   real robot. Nothing failed then either; the sim was simply a different
   vehicle. Gazebo still was.

Key Changes:
1. Rear axle (gazebo/runtime/robot_description/wro_robot.urdf.xacro)
* Adds rear_{left,right}_steering links and revolute joints, and re-parents
  the rear wheels onto them -- adding the hinge alone would look right in a
  diff and change nothing in simulation.
* Each rear joint mimics its OWN front counterpart at -rear_steer_ratio.
  A mimic constraint, not a controller: the stock gz-sim AckermannSteering
  plugin steers one axle by construction, and expressing the relationship as
  a physics constraint means the axles cannot drift out of phase and no
  extra node has to publish the rear angle. SDFormat documents its mimic
  multiplier/offset as matching the URDF tag's.
* Emitted through a xacro macro, so left and right cannot diverge.
* Fixes the three illegal `--` comment sequences.

2. Ratio plumbing (gazebo/generator/internal/robotconfig/generate.go)
* rear_steer_ratio reached the Go constants as RobotRearSteerRatio but was
  never emitted into robot_properties.gen.xacro, so the URDF had no way to
  express counter-phase except by restating 1.0 as a literal. Now emitted;
  a chassis rebuilt front-steer-only pins the rear wheels straight from
  robot.toml without touching the URDF.

3. Test coverage (platform/robot/tests/unit/, pixi.toml)
* test_gazebo_urdf_matches_chassis.py expands the description and checks the
  rear axle steers, the wheels hang off it, the mimic is negative and
  tracks robot.toml, and the axle geometry still matches RobotSpecs.
* Adds ros-kilted-xacro to the dev feature. `import xacro` in dev resolved
  to an EMPTY namespace package (__file__ None, no process_file), so an
  importorskip guard was satisfied and the test would have skipped in CI --
  the same silence that let the unparseable URDF sit here in the first place.

Verification:
* xacro now expands: 13 links, 12 joints. Rear steering joints carry
  MIMIC front_{side}_steering_joint x-1.0; rear wheels parent to
  rear_{side}_steering.
* HEAD's version fails to expand at all -- confirmed directly, not inferred.
* 11 new tests pass; all 11 ERROR against the pre-fix URDF, so they fail for
  the right reason rather than passing vacuously.
* NOT run in Gazebo. gz does not launch on this Windows host (the gz conda
  packages ship .bat-only activation, so GZ_CONFIG_PATH is never set), which
  is also why these defects survived. The mimic constraint needs a Linux run
  to confirm the physics engine honours it.

File: platform/gazebo/runtime/robot_description/robot_properties.gen.xacro (robot description, xacro)
@@ -11,4 +11,5 @@
   <xacro:property name="track_width" value="0.1675"/>
   <xacro:property name="max_steering_angle" value="0.9599310885968813"/>
+  <xacro:property name="rear_steer_ratio" value="1.0"/>
   <!-- Wheel properties -->
   <xacro:property name="wheel_radius" value="0.035"/>

File: platform/gazebo/runtime/robot_description/wro_robot.urdf.xacro (robot description, xacro)
@@ -1,5 +1,5 @@
 <?xml version="1.0"?>
 <robot name="wro_robot" xmlns:xacro="http://www.ros.org/wiki/xacro">
-  <!-- Chassis/Ackermann/wheel/sensor-mount properties -- generated from
+  <!-- Chassis/Ackermann/wheel/sensor-mount properties, generated from
        platform/shared/config/robot.toml, see robot_properties.gen.xacro. -->
   <xacro:include filename="robot_properties.gen.xacro"/>
@@ -113,19 +113,50 @@
     <axis xyz="0 1 0"/>
   </joint>
-  <!-- ====== REAR WHEELS (Drive) ====== -->
-  <xacro:wheel_link name="rear_left_wheel"/>
-  <joint name="rear_left_wheel_joint" type="continuous">
-    <parent link="base_link"/>
-    <child link="rear_left_wheel"/>
-    <origin xyz="${-half_wheelbase} ${half_track} 0" rpy="0 0 0"/>
-    <axis xyz="0 1 0"/>
-  </joint>
-  <xacro:wheel_link name="rear_right_wheel"/>
-  <joint name="rear_right_wheel_joint" type="continuous">
-    <parent link="base_link"/>
-    <child link="rear_right_wheel"/>
-    <origin xyz="${-half_wheelbase} ${-half_track} 0" rpy="0 0 0"/>
-    <axis xyz="0 1 0"/>
-  </joint>
+  <!-- ====== REAR WHEELS (Drive + counter-phase steering) ====== -->
+  <!-- The rear axle STEERS, opposite the front and by the same amount at
+       rear_steer_ratio=1.0. Confirmed on the real chassis 2026-07-25 and
+       re-verified by hand 2026-08-15; src/simulation/kinematics.py has
+       integrated it since, and tests/unit/test_kinematics_4ws.py guards it.
+       This file did not, until 2026-08-22: the rear wheels bolted straight to
+       base_link as plain drive joints, so Gazebo was a front-steer car. That
+       is not a cosmetic difference. Counter-phase moves the instantaneous
+       centre of rotation from the rear axle to the chassis centre
+       (L_eff = wheelbase / (1 + rear_steer_ratio)), so the robot yaws TWICE as
+       fast for a given steering angle: the exact discrepancy that was found
+       and fixed on the headless side, where it had silently made every gain
+       tuned against the sim hotter on the real robot.
+       Driven by a mimic constraint rather than a controller: the stock
+       gz-sim AckermannSteering plugin below steers ONE axle by construction,
+       and mimic expresses "follower = multiplier * leader" as a physics
+       constraint, so the rear angle cannot drift out of phase with the front
+       and no extra node has to publish it. SDFormat's mimic multiplier/offset
+       are documented to match the URDF mimic tag's. -->
+  <xacro:macro name="rear_steering_assembly" params="side y_sign">
+    <xacro:steering_link name="rear_${side}_steering"/>
+    <joint name="rear_${side}_steering_joint" type="revolute">
+      <parent link="base_link"/>
+      <child link="rear_${side}_steering"/>
+      <origin xyz="${-half_wheelbase} ${y_sign * half_track} 0" rpy="0 0 0"/>
+      <axis xyz="0 0 1"/>
+      <limit lower="${-max_steering_angle}" upper="${max_steering_angle}" effort="10" velocity="3.0"/>
+      <!-- Negative: counter-phase. rear_steer_ratio comes from robot.toml via
+           robot_properties.gen.xacro, so a chassis rebuilt front-steer-only
+           (ratio 0.0) pins the rear wheels straight without editing this file. -->
+      <mimic joint="front_${side}_steering_joint" multiplier="${-rear_steer_ratio}" offset="0"/>
+    </joint>
+    <xacro:wheel_link name="rear_${side}_wheel"/>
+    <!-- Parented to the steering link, not base_link: that re-parenting is
+         what actually makes the wheel turn. The AckermannSteering plugin still
+         drives this joint for propulsion; it is unaffected by the extra hinge
+         above it. -->
+    <joint name="rear_${side}_wheel_joint" type="continuous">
+      <parent link="rear_${side}_steering"/>
+      <child link="rear_${side}_wheel"/>
+      <origin xyz="0 0 0" rpy="0 0 0"/>
+      <axis xyz="0 1 0"/>
+    </joint>
+  </xacro:macro>
+  <xacro:rear_steering_assembly side="left" y_sign="1"/>
+  <xacro:rear_steering_assembly side="right" y_sign="-1"/>
   <!-- ====== SENSORS ====== -->
   <!-- Camera (RPi Camera 3 Wide: 102 deg HFOV, 1536x864) -->
@@ -213,5 +244,5 @@
     <!-- z = chassis_height + lidar_mount_z = 0.12: matches static_tfs.launch.py / the Go
          SDF generator's RobotHeight + RobotLidarMountZOffset. Previously chassis_height/2
-         + 0.025 = 0.075 here only -- a pre-existing drift from those other two sources,
+         + 0.025 = 0.075 here only, a pre-existing drift from those other two sources,
          found and fixed alongside the mount-offset measurements (see
          platform/robot/docs/robot-physical-constants.md). lidar_mount_z is now generated
@@ -273,5 +304,5 @@
     <child link="imu_link"/>
     <!-- z = imu_mount_z = 0.01: matches static_tfs.launch.py / the Go SDF generator's
-         RobotImuMountZOffset. Was hardcoded to 0 here only -- a pre-existing drift from
+         RobotImuMountZOffset. Was hardcoded to 0 here only, a pre-existing drift from
          those other two sources, found while consolidating the mount-offset source of
          truth into platform/shared/config/robot.toml. -->

Commit message: fix(robot): the LIDAR scan plane is 0.08 m off the floor, not the 0.12 the config derived
The repo derived the scan plane as chassis.height (0.10) + lidar.mount_z_offset
(+0.02) = 0.12 m. The beam MEASURES ~0.08 m. The offset is negative: the unit
is recessed, not stacked 20 mm above the chassis top as the field claimed.

Cause:
Nothing cross-checked the derived height against the track it has to see. In
track.toml EVERY object on the field is 0.10 m tall -- wall.height, the pillars
and the blocks alike -- so at 0.12 m the beam clears the entire course and the
robot is blind. It plainly is not: over run_20260907_031019 the +/-90 deg rays
read p10 0.20 / median 0.58 / p90 1.79 m in a 1.0 m corridor, which is the
walls, exactly where they are.

This is load-bearing for REASONING, not just for TF. From the wrong 0.12 it
follows that the LIDAR cannot see a 0.10 m traffic sign at all -- a conclusion
I reached and nearly acted on, with an empirical result that appeared to
confirm it (at the committed sign's bearing only 14.2% of returns were
consistent with the sign and 48.4% landed beyond it). That number is real but
it is not beam geometry; the same argument would make wall-following
impossible. It is far better explained by believed sign positions being wrong,
given the known phantoms and ~2.7x track duplication. At the true 0.08 m the
beam crosses a 0.10 m sign 2 cm below its top, on the body.

Key Changes:
1. Config (platform/shared/config/robot.toml)
* lidar.mount_z_offset 0.02 -> -0.02, with the measurement and the
  wall-return evidence recorded on the field.

2. Gazebo description (platform/gazebo/runtime/robot_description/)
* robot_properties.gen.xacro lidar_mount_z 0.02 -> -0.02. The file is
  hand-maintained (its generator was removed 2026-09-03), so it does not
  follow robot.toml on its own.
* wro_robot.urdf.xacro: the joint origin already derives correctly from
  chassis_height + lidar_mount_z; only its "= 0.12" comment was stale.

3. Visualizer (platform/robot/src/simulation/live_visualizer/visualizer.py)
* Stale "= 0.12" comment corrected. The marker itself reads from config.

Verification:
* RobotSpecs.HEIGHT + LIDAR_MOUNT_Z_OFFSET now evaluates to exactly 0.080.
* static_tfs.launch.py and the visualizer marker both derive from that sum, so
  they follow without edits; the xacro property and three comments were the
  only hand-copied duplicates left.
* Unaffected by the negative value: no validator constrains mount_z_offset to
  be positive (robot_constants.py declares it a bare float).
* tests -k constant: 77 passed, 1 pre-existing failure
  (test_lidar_max_range_safety_margin, about LIDAR_MAX_RANGE vs the hardware
  max, untouched here). tests -k lidar and -k geometry cannot run at all on
  this machine -- they die with a Windows access violation that reproduces at
  clean HEAD.

Follow-on this unblocks: LIDAR picks up persistent pillar-shaped clusters at a
median 1.10-1.30 m (p90 ~1.87 m) where the camera's median detection range is
0.70 m, so it can propose obstacle candidates in the band where vision goes
blind. Precision is the open question -- 30-110 persistent tracks per run
against ~8 real signs.

File: platform/gazebo/runtime/robot_description/robot_properties.gen.xacro (robot description, xacro)
@@ -21,5 +21,7 @@
   <!-- Sensor mount offsets -->
   <xacro:property name="lidar_mount_x" value="0.1222"/>
-  <xacro:property name="lidar_mount_z" value="0.02"/>
+  <!-- NEGATIVE: the unit is recessed, not stacked on the chassis top. The beam
+       MEASURES ~0.08 m off the floor (2026-09-07), so chassis_height + this = 0.08. -->
+  <xacro:property name="lidar_mount_z" value="-0.02"/>
   <xacro:property name="lidar_mount_yaw_offset_deg" value="180.0"/>
   <xacro:property name="imu_mount_z" value="0.01"/>

File: platform/gazebo/runtime/robot_description/wro_robot.urdf.xacro (robot description, xacro)
@@ -242,5 +242,5 @@
     <parent link="base_link"/>
     <child link="lidar_link"/>
-    <!-- z = chassis_height + lidar_mount_z = 0.12: matches static_tfs.launch.py / the Go
+    <!-- z = chassis_height + lidar_mount_z = 0.08: matches static_tfs.launch.py / the Go
          SDF generator's RobotHeight + RobotLidarMountZOffset. Previously chassis_height/2
          + 0.025 = 0.075 here only, a pre-existing drift from those other two sources,

Commit message: fix(sim): correct camera mount to measured pose (z=0.20 m, ~10 deg down)

File: platform/gazebo/runtime/robot_description/robot_properties.gen.xacro (robot description, xacro)
@@ -27,5 +27,5 @@
   <xacro:property name="imu_mount_z" value="0.01"/>
   <xacro:property name="camera_mount_x" value="0.1222"/>
-  <xacro:property name="camera_mount_z" value="0.16"/>
-  <xacro:property name="camera_mount_pitch" value="0.5236"/>
+  <xacro:property name="camera_mount_z" value="0.20"/>
+  <xacro:property name="camera_mount_pitch" value="0.1745"/>
 </robot>
